Commit message: add three new models

File: models/dual_v2_1_no_gripper/robot.urdf (robot description, URDF)
Before this commit: robot dual_v2_1, 24 links, 23 joints
Links:
- link arm_L2_l: mass 0.72275 -> 0.722746273788613
- link arm_L2_r: mass 0.72275 -> 0.722746273788613
- link arm_L3_l: mass 1.7397 -> 1.73968859476709
- link arm_L3_r: mass 1.7397 -> 1.73968859476709
- link arm_L4_l: mass 1.299 -> 1.29895883494625
- link arm_L4_r: mass 1.299 -> 1.29895883494625
- link arm_L5_l: mass 0.94391 -> 0.943914533169422
- link arm_L5_r: mass 0.94391 -> 0.943914533169422
- link arm_L6_l: mass 0.87461 -> 0.874611215710047
- link arm_L6_r: mass 0.87461 -> 0.874611215710047
- link arm_L7_l: mass 0.75543 -> 0.755421642189138
- link arm_L7_r: mass 0.75543 -> 0.755421642189138

File: models/dual_v2_2_no_gripper/robot.urdf (robot description, URDF)
Before this commit: robot dual_v2_2, 26 links, 25 joints
Joints:
- joint H1: axis (none) -> 0 0 1; limit (none) -> lower=0 upper=0 effort=0 velocity=0; type fixed -> revolute
- joint H2: axis (none) -> 0 0 1; limit (none) -> lower=0 upper=0 effort=0 velocity=0; type fixed -> revolute
- joint S1: axis (none) -> 0 0 1; limit (none) -> lower=0 upper=0 effort=0 velocity=0; type fixed -> revolute
- joint S2: axis (none) -> 0 0 1; limit (none) -> lower=0 upper=0 effort=0 velocity=0; type fixed -> revolute
- joint S3: axis (none) -> 0 0 1; limit (none) -> lower=0 upper=0 effort=0 velocity=0; type fixed -> revolute
- joint S4: axis (none) -> 0 0 1; limit (none) -> lower=0 upper=0 effort=0 velocity=0; type fixed -> revolute

File: models/spark2_v1/robot.urdf (robot description, URDF)
Before this commit: robot arm_v1, 9 links, 8 joints
Joints:
- joint arm_J1: origin xyz=0.000000000 0.000000000 0.0962      rpy=0.000000000 0.000000000 0.000000000 -> xyz=0.000000000 0.000000000 0.0962 rpy=0.000000000 0.000000000 0.000000000
- joint arm_J2: origin xyz= 0.0965       0.000000000  0.000000000 rpy= -1.57079632  -1.57079632  0.000000000 -> xyz=0.0965 0.000000000 0.000000000 rpy=-1.57079632 -1.57079632 0.000000000
- joint arm_J3: origin xyz= 0.3465       0.000000000  0.000000000 rpy= 0.000000000  0.000000000  0.000000000 -> xyz=0.3465 0.000000000 0.000000000 rpy=0.000000000 0.000000000 0.000000000
- joint arm_J4: origin xyz= 0.15         0.000000000  0.000000000 rpy= 0.000000000  0.000000000  0.000000000 -> xyz=0.15 0.000000000 0.000000000 rpy=0.000000000 0.000000000 0.000000000
- joint arm_J5: origin xyz= 0.000000000  0.0965      0.000000000 rpy= -1.57079632  -1.57079632  0.000000000 -> xyz=0.000000000 0.0965 0.000000000 rpy=-1.57079632 -1.57079632 0.000000000
- joint arm_J6: origin xyz= 0.000000000  0.185  0.000000000 rpy= -1.57079632  0.000000000  0.000000000 -> xyz=0.000000000 0.185 0.000000000 rpy=-1.57079632 0.000000000 0.000000000
